File: RF_Related/Pol Switch/polarization_switch_mid_redo.sch (EAGLE design)
At the start: 61 parts, among them IC1 VLPR-24-858-2, IC10 ADP-2-1+_MINICIRCUITS, IC11 ADP-2-1+_MINICIRCUITS, IC12 QCV-151+, IC13 MAX8878EUK28+T, IC14 SN74LVC2G17DBVT, IC15 SN74LVC2G17DBVT, IC2 VLPR-24-858-2, IC3 HSWA2-30DR+, IC4 VLPR-24-858-2, IC5 HSWA2-30DR+, IC6 HSWA2-30DR+, IC7 HSWA2-30DR+, IC8 PHA-13LN+, IC9 PHA-13LN+, J1 M20-9730645, J2 171856-0002, X3 SMA-142-0701-801/806, X4 SMA-142-0701-801/806, X5 SMA-142-0701-801/806

Commit message: made a new pol switch board with jumper pads. do I need that resistor row? backing up now
Parts:
- removed C13: 10e-6, rcl:C-USC0603
- removed C14: 1e-9, rcl:C-USC0603
- removed X4: SMA-142-0701-801/806, sma-flange_375mils:SMA-142-0701-801/806
- added R4: 0, rcl:R-US_R1206
- added X2: SMA-142-0701-801/806, sma-flange_375mils:SMA-142-0701-801/806
- renumbered X5 to X1
Connections:
- removed net N$18: IC11.PORT_2, IC6G$1.RF1
- removed net N$23: IC11.PORT_1, IC5G$1.RF1
- new net N$10: IC11.PORT_2, R4.2
- new net N$11: IC11.PORT_1, IC6G$1.RF1
- new net N$12: IC5G$1.RF1, R4.1
- net GND: now also X2.2; no longer C13.1, C14.1, X4.2
- net N$29: now also X2.1; no longer X3.1
- net N$31: now also X3.1; no longer X4.1
- net N$36: no longer C13.2, C14.2
- net N$4: now also IC10.PORT_2; no longer IC10.PORT_1
- net N$7: now also IC10.PORT_1; no longer IC10.PORT_2
Other:
- moved on the sheet: X3
